Commit message: link names update joint pose update

File: urdf/turtlebot3_waffle.urdf (robot description, URDF)
Before this commit: robot turtlebot3_waffle, 13 links, 12 joints
Joints:
- joint camera_rgb_joint: origin xyz=0.005 0.018 0.013 rpy=0 0 0 -> xyz=0.005 0.018 0.013 rpy=-1.57 0 -1.57; parent camera_link -> realsense_link
- joint realsense_depth_joint: origin xyz=0.005 0.028 0.013 rpy=0 0 0 -> xyz=0.005 0.028 0.013 rpy=-1.57 0 -1.57; parent camera_link -> realsense_link
